Commit message: クローラで動けるようにした

File: assets/zx120/zx120.urdf (robot description, URDF)
Before this commit: robot zx120, 7 links, 6 joints
Links:
- added link left_front_wheel_link, mass 10; collision cylinder length=0.5 radius=0.35
- added link left_middle_wheel_link, mass 10; collision cylinder length=0.5 radius=0.35
- added link left_rear_wheel_link, mass 10; collision cylinder length=0.5 radius=0.35
- added link right_front_wheel_link, mass 10; collision cylinder length=0.5 radius=0.35
- added link right_middle_wheel_link, mass 10; collision cylinder length=0.5 radius=0.35
- added link right_rear_wheel_link, mass 10; collision cylinder length=0.5 radius=0.35
- link track_link: mass 10 -> 1
Joints:
- added joint left_front_wheel_joint: type continuous, parent base_link, child left_front_wheel_link, origin xyz=1.284131 1 0.35 rpy=-1.5707963267948966 0 0, axis 0 0 1
- added joint left_middle_wheel_joint: type continuous, parent base_link, child left_middle_wheel_link, origin xyz=-0.155869 1 0.35 rpy=-1.5707963267948966 0 0, axis 0 0 1
- added joint left_rear_wheel_joint: type continuous, parent base_link, child left_rear_wheel_link, origin xyz=-1.595869 1 0.35 rpy=-1.5707963267948966 0 0, axis 0 0 1
- added joint right_front_wheel_joint: type continuous, parent base_link, child right_front_wheel_link, origin xyz=1.284131 -1 0.35 rpy=-1.5707963267948966 0 0, axis 0 0 1
- added joint right_middle_wheel_joint: type continuous, parent base_link, child right_middle_wheel_link, origin xyz=-0.155869 -1 0.35 rpy=-1.5707963267948966 0 0, axis 0 0 1
- added joint right_rear_wheel_joint: type continuous, parent base_link, child right_rear_wheel_link, origin xyz=-1.595869 -1 0.35 rpy=-1.5707963267948966 0 0, axis 0 0 1

Commit message: remove unused assets, クローラの動きをスムーズにするため1cm車体を浮かす

File: assets/zx120/zx120.urdf (robot description, URDF)
Before this commit: robot zx120, 13 links, 12 joints
Joints:
- joint base_joint: origin (none) -> xyz=0 0 0.01 rpy=0 0 0
